File: micro.sch (KiCad schematic (older format))
At the start: 18 parts, among them J1 RJ45-MAG, P1 CONN_4, P2 CONN_4, P3 CONN_2, SW1 SW_PUSH, U1 7805, U2 7833

Commit message: borrando archivos viejos
Parts:
- C1: value 10u -> 0.33u
- C3: value 10u -> 0.1u
Changed lines of the file:
@@
-EESchema Schematic File Version 2  date dom 17 feb 2013 13:57:08 ART
+EESchema Schematic File Version 2  date lun 18 feb 2013 15:53:11 ART
 LIBS:w_connectors
 LIBS:micro-cache
@@
 Sheet 1 1
 Title "uControlador"
-Date "17 feb 2013"
+Date "18 feb 2013"
 Rev "1.0"
 Comp "Seminario de Sistemas Embebidos - FIUBA"
@@
 P 4050 3400
 F 0 "C3" H 4100 3500 50  0000 L CNN
-F 1 "10u" H 4100 3300 50  0000 L CNN
+F 1 "0.1u" H 4100 3300 50  0000 L CNN
 	1    4050 3400
 	1    0    0    -1
@@
 P 1750 3400
 F 0 "C1" H 1800 3500 50  0000 L CNN
-F 1 "10u" H 1800 3300 50  0000 L CNN
+F 1 "0.33u" H 1800 3300 50  0000 L CNN
 	1    1750 3400
 	1    0    0    -1
